File: v1/nfc-pn532.brd (EAGLE design)
At the start: 101 x 50 mm, 53 parts, among them U1 PN532, U2 MIC5225-3.3V, X1 B7B-PH-SM4-TB, Y1 27.12MHz

Commit message: updating schematic
Parts:
- added R7: 10K, microbuilder:0805-NO
Connections:
- net RSTPD_N: now also R7.2
- net VDD: now also R7.1
Routing:
- net GND: track 94.0 -> 92.2 mm
- net VDD: track 77.0 -> 78.6 mm
- net RSTPD_N: track 6.33 -> 7.04 mm
Changed lines of the file:
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@@
 <attribute name="VALUE" x="77.55" y="44.505" size="1.016" layer="27" rot="R180" align="bottom-right"/>
+</element>
+<element name="R7" library="microbuilder" package="0805-NO" value="10K" x="91.6" y="35.55" smashed="yes" rot="R270">
+<attribute name="NAME" x="91.373" y="33.618" size="0.8128" layer="25" ratio="18" rot="R270"/>
+<attribute name="VALUE" x="90.838" y="33.518" size="0.4064" layer="27" ratio="10" rot="R270"/>
 </element>
 </elements>
@@
 <wire x1="89.964" y1="29.205" x2="89.715" y2="29.718" width="0.2032" layer="1"/>
 <wire x1="89.964" y1="36.576" x2="88.29" y2="38.25" width="0.3048" layer="1"/>
-<wire x1="89.964" y1="36.576" x2="89.964" y2="35.616" width="0.3048" layer="1"/>
+<wire x1="89.964" y1="36.576" x2="89.964" y2="36.55" width="0.3048" layer="1"/>
+<wire x1="89.964" y1="36.55" x2="89.964" y2="35.616" width="0.3048" layer="1"/>
 <wire x1="89.964" y1="35.616" x2="89.908" y2="35.56" width="0.3048" layer="1"/>
 <via x="89.908" y="31.662" extent="1-16" drill="0.5"/>
@@
 <wire x1="93.1" y1="10.15" x2="93.1" y2="20.75" width="0.2032" layer="16"/>
 <wire x1="93.1" y1="20.75" x2="95.718" y2="23.368" width="0.2032" layer="16"/>
+<contactref element="R7" pad="1"/>
+<wire x1="91.6" y1="36.5" x2="90.014" y2="36.5" width="0.2032" layer="1"/>
+<wire x1="90.014" y1="36.5" x2="89.964" y2="36.55" width="0.2032" layer="1"/>
 </signal>
 <signal name="GND">
@@
 <wire x1="94.22" y1="38.23268125" x2="94.22" y2="38.728" width="0.508" layer="1"/>
 <wire x1="95.24" y1="37.21268125" x2="94.22" y2="38.23268125" width="0.508" layer="1"/>
-<wire x1="92.621" y1="32.785" x2="92.621" y2="34.748" width="0.2032" layer="1"/>
-<wire x1="92.621" y1="34.748" x2="94.0422625" y2="34.748" width="0.2032" layer="1"/>
 <wire x1="94.0422625" y1="34.748" x2="94.0676625" y2="34.7226" width="0.2032" layer="1"/>
 <wire x1="96.5283375" y1="34.7226" x2="96.6037375" y2="34.798" width="0.2032" layer="1"/>
 <wire x1="96.6037375" y1="34.798" x2="97.203" y2="34.798" width="0.2032" layer="1"/>
 <wire x1="94.0676625" y1="34.7226" x2="96.5283375" y2="34.7226" width="0.254" layer="1"/>
-<via x="91.659" y="35.202" extent="1-16" drill="0.5"/>
 <wire x1="77.899" y1="36.83" x2="74.47" y2="33.401" width="0.2032" layer="16"/>
 <via x="74.47" y="33.401" extent="1-16" drill="0.3937"/>
@@
 <wire x1="92.734" y1="24.62" x2="92.092" y2="23.978" width="0.254" layer="1"/>
 <wire x1="92.092" y1="23.978" x2="92.079" y2="23.978" width="0.254" layer="1"/>
+<via x="93" y="34.2" extent="1-16" drill="0.3937"/>
+<wire x1="92.621" y1="32.785" x2="92.621" y2="33.78995" width="0.2032" layer="1"/>
+<wire x1="92.621" y1="33.78995" x2="92.6548" y2="33.82375" width="0.2032" layer="1"/>
+<wire x1="92.6548" y1="33.82375" x2="92.6548" y2="33.8548" width="0.2032" layer="1"/>
+<wire x1="92.6548" y1="33.8548" x2="93" y2="34.2" width="0.2032" layer="1"/>
 </signal>
 <signal name="N$1">
@@
 <signal name="RSTPD_N">
 <contactref element="U1" pad="38"/>
-<wire x1="91.484" y1="32.616" x2="90.55" y2="33.55" width="0.2032" layer="1"/>
-<wire x1="91.484" y1="27.61" x2="91.484" y2="32.616" width="0.2032" layer="1"/>
+<contactref element="R7" pad="2"/>
+<wire x1="91.484" y1="34.484" x2="91.6" y2="34.6" width="0.2032" layer="1"/>
+<wire x1="91.484" y1="27.61" x2="91.484" y2="34.484" width="0.2032" layer="1"/>
 </signal>
 </signals>
