File: v1/nfc-pn532.sch (EAGLE design)
At the start: 53 parts, among them U1 PN532, U2 MIC5225-3.3V, X1 B7B-PH-SM4-TB, Y1 27.12MHz

Commit message: updating schematic
Parts:
- added R7: 10K, microbuilder:RESISTOR0805_NOOUTLINE
Connections:
- net RSTPD_N: now also R7.2
- net VDD: now also R7.1
Other:
- note added: "Molex 55460-0772"
Changed lines of the file:
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@@
 <part name="U$6" library="microbuilder" deviceset="VIN" device=""/>
 <part name="U$23" library="microbuilder" deviceset="GND" device=""/>
+<part name="R7" library="microbuilder" deviceset="RESISTOR" device="0805_NOOUTLINE" value="10K"/>
+<part name="U$1" library="microbuilder" deviceset="VDD" device=""/>
 </parts>
 <sheets>
@@
 1008CS-561</text>
 <text x="152.4" y="215.9" size="1.778" layer="97">10uF removed in v1.6</text>
+<text x="307.34" y="124.46" size="1.778" layer="91">Molex 55460-0772</text>
 </plain>
 <instances>
@@
 <instance part="U$23" gate="G$1" x="307.34" y="154.94" smashed="yes" rot="R180">
 <attribute name="VALUE" x="308.864" y="157.48" size="1.27" layer="96" rot="R180"/>
+</instance>
+<instance part="R7" gate="G$1" x="200.66" y="172.72" smashed="yes" rot="R180">
+<attribute name="NAME" x="203.2" y="170.688" size="1.27" layer="95" font="vector" rot="R180"/>
+<attribute name="VALUE" x="203.2" y="175.895" size="1.27" layer="96" font="vector" rot="R180"/>
+</instance>
+<instance part="U$1" gate="G$1" x="210.82" y="172.72" smashed="yes" rot="R270">
+<attribute name="VALUE" x="211.836" y="174.244" size="1.27" layer="96" rot="R270"/>
 </instance>
 </instances>
@@
 <wire x1="210.82" y1="73.66" x2="215.9" y2="73.66" width="0.1524" layer="91"/>
 <junction x="210.82" y="73.66"/>
+</segment>
+<segment>
+<pinref part="R7" gate="G$1" pin="1"/>
+<pinref part="U$1" gate="G$1" pin="VDD"/>
+<wire x1="205.74" y1="172.72" x2="208.28" y2="172.72" width="0.1524" layer="91"/>
 </segment>
 </net>
@@
 <pinref part="U1" gate="G$1" pin="RSTPD_N"/>
 <wire x1="190.5" y1="162.56" x2="190.5" y2="170.18" width="0.1524" layer="91"/>
-<label x="190.5" y="170.18" size="1.4224" layer="95" rot="R90" xref="yes"/>
-</segment>
-</net>
+<pinref part="R7" gate="G$1" pin="2"/>
+<wire x1="195.58" y1="172.72" x2="190.5" y2="172.72" width="0.1524" layer="91"/>
+<wire x1="190.5" y1="172.72" x2="190.5" y2="170.18" width="0.1524" layer="91"/>
+</segment>
+</net>
